Commit message: Finished URDF of soliro but not yet with correct mass and inertia

File: rotors_description/urdf/soliro.xacro (robot description, xacro)
@@ -9,8 +9,8 @@
     <xacro:property name="use_mesh_file_rotor_unit" value="true"/>
     <!-- TODO change add meshes to package -->
-    <xacro:property name="mesh_file_core" value="package://rotors_description/meshes/soliro/main.stl"/>
-    <xacro:property name="mesh_file_core_collision" value="package://rotors_description/meshes/soliro/main.stl"/>
-    <xacro:property name="mesh_file_right_wing" value="package://rotors_description/meshes/soliro/soliro_wing_right.stl"/>
-    <xacro:property name="mesh_file_right_motor" value="package://rotors_description/meshes/soliro/motor_right.stl"/>
+    <xacro:property name="mesh_soliro_base" value="package://rotors_description/meshes/soliro/soliro_body.stl"/>
+    <xacro:property name="mesh_soliro_base_collision" value="package://rotors_description/meshes/soliro/soliro_body.stl"/>
+    <xacro:property name="mesh_soliro_wing" value="package://rotors_description/meshes/soliro/soliro_wing_right.stl"/>
+    <xacro:property name="mesh_soliro_motor_unit" value="package://rotors_description/meshes/soliro/motor_unit.stl"/>
     <xacro:property name="mass_core" value="3.13"/>    <!-- [kg] -->
     <xacro:property name="mass_tilt_unit" value="0.277"/>    <!-- [kg] -->
@@ -32,10 +32,10 @@
         <!-- [kg m^2] [kg m^2] [kg m^2] [kg m^2] [kg m^2] [kg m^2] -->
     </xacro:property>
-    <!-- Body Interia / CoM Offset -->
+    <!-- Body Inertia / CoM Offset -->
     <xacro:property name="body_inertia_origin">
         <!-- <origin xyz="0.03 0 0.01" /> -->
         <origin xyz="0.0 0.0 0.0" />
     </xacro:property>
-    <!-- Rotor unit inertia without the propellor. -->
+    <!-- Rotor unit inertia without the propeller. -->
     <xacro:property name="tilt_unit_inertia">
         <inertia ixx="0.00034257" ixy="0" ixz="0" iyy="0.0013205" iyz="0" izz="0.0010037"/>
@@ -53,12 +53,11 @@
             body_height="${body_height}"
             use_mesh_file="${use_mesh_file_core}"
-            mesh_file="${mesh_file_core}"
-            collision_mesh_file="${mesh_file_core_collision}">
+            mesh_file="${mesh_soliro_base}"
+            collision_mesh_file="${mesh_soliro_base_collision}">
         <xacro:insert_block name="body_origin"/>
         <xacro:insert_block name="body_inertia"/>
         <xacro:insert_block name="body_inertia_origin"/>
     </xacro:soliro_base_macro>
-    <!-- TODO Instantiate left and right wing -->
-    <!-- right -->
+    <!-- Right wing unit-->
     <xacro:wing_unit
             robot_namespace="${namespace}"
@@ -69,10 +68,35 @@
             rotor_offset_top="${rotor_offset_top}"
             wing_number="0"
-            mesh="propeller"
-            mesh_tilt_wing="${mesh_file_right_wing}"
+            mesh_tilt_wing="${mesh_soliro_wing}"
+            mesh_motor_unit="${mesh_soliro_motor_unit}"
             color="Black">
-        <origin xyz="0 -${arm_length} 0" rpy="0 0 4.71238898038"/>
+        <origin xyz="0 0 0" rpy="0 0 0"/>
         <xacro:insert_block name="rotor_inertia" />
     </xacro:wing_unit>
-    <!-- TODO Instantiate rear tilt rotor -->
+    <!-- Left wing unit-->
+    <xacro:wing_unit
+            robot_namespace="${namespace}"
+            direction="ccw"
+            parent="${tilt_unit_parent}"
+            mass_rotor="${mass_rotor}"
+            mass_tilt_unit="${mass_tilt_unit}"
+            rotor_offset_top="${rotor_offset_top}"
+            wing_number="1"
+            mesh_tilt_wing="${mesh_soliro_wing}"
+            mesh_motor_unit="${mesh_soliro_motor_unit}"
+            color="Black">
+        <origin xyz="0 0 0" rpy="0 0 0"/>
+        <xacro:insert_block name="rotor_inertia" />
+    </xacro:wing_unit>
+    <!-- Rear actuation unit -->
+    <xacro:rear_rotor
+            robot_namespace="${namespace}"
+            direction="ccw"
+            parent="${tilt_unit_parent}"
+            mass_rotor="${mass_rotor}"
+            rotor_offset_top="0.05"
+            color="Black">
+        <origin xyz="-0.7845 0 0.0325" rpy="0 0 0"/>
+        <xacro:insert_block name="rotor_inertia" />
+    </xacro:rear_rotor>
 </robot>

File: rotors_description/urdf/soliro_actuators.xacro (robot description, xacro)
@@ -1,3 +1,146 @@
 <?xml version="1.0"?>
 <robot name="$(arg mav_name)" xmlns:xacro="http://ros.org/wiki/xacro">
+    <!-- Motor Parameters -->
+    <xacro:property name="motor_constant" value="${7.2e-06}"/>    <!-- [kg m/s^2] -->
+    <xacro:property name="moment_constant" value="0.015"/>    <!-- [m] -->
+    <xacro:property name="time_constant_up" value="0.0125"/>    <!-- [s] -->
+    <xacro:property name="time_constant_down" value="0.025"/>    <!-- [s] -->
+    <xacro:property name="min_rot_velocity" value="100"/>
+    <xacro:property name="max_rot_velocity" value="1700"/>    <!-- [rad/s] --> <!-- Velocity to produce 1 kg thrust -->
+    <xacro:property name="rotor_drag_coefficient" value="${8.06428e-05}"/>
+    <xacro:property name="rolling_moment_coefficient" value="0.000001"/>
+    <!-- Relationship between the p, d gain and the closed-loop dynamics behaviour of the system:
+    It behaves like a second-order system in the frequency domain: Y(s) = U(s)*(ds + p)/(Is**2 + ds + p)
+    Y(s) is the Laplace transform of the actual tilt motor angle and U(s) is the one of the tilt motor angle command, p and d are the gains, I is the inertia of the link.
+    The pid gain set here corresponds to p = 1200, i = 1000, d =500 on the firmware.
+     -->
+    <xacro:property name="tilt_control_mode" value="position"/>
+    <xacro:property name="p_gain" value="0.11"/>
+    <xacro:property name="i_gain" value="0.0"/>
+    <xacro:property name="d_gain" value="0.1"/>
+    <xacro:property name="servo_zero_offset" value="0.0"/>
+    <!-- Add motors. -->
+    <gazebo>
+        <plugin name="multimotor_plugin" filename="librotors_gazebo_multimotor_plugin.so">
+            <robotNamespace>$(arg mav_name)</robotNamespace>
+            <rotors>
+                <rotor>
+                    <jointName>rotor_0_joint</jointName>
+                    <linkName>rotor_0</linkName>
+                    <spinDirection>ccw</spinDirection>
+                    <timeConstantUp>${time_constant_up}</timeConstantUp>
+                    <timeConstantDown>${time_constant_down}</timeConstantDown>
+                    <minRotVelocity>${min_rot_velocity}</minRotVelocity>
+                    <maxRotVelocity>${max_rot_velocity}</maxRotVelocity>
+                    <thrustConstant>${motor_constant}</thrustConstant>
+                    <momentConstant>${moment_constant}</momentConstant>
+                    <rotorDragCoefficient>${rotor_drag_coefficient}</rotorDragCoefficient>
+                    <rollingMomentCoefficient>${rolling_moment_coefficient}</rollingMomentCoefficient>
+                    <rotorVelocitySlowdownSim>${rotor_velocity_slowdown_sim}</rotorVelocitySlowdownSim>
+                </rotor>
+                <rotor>
+                    <jointName>rotor_1_joint</jointName>
+                    <linkName>rotor_1</linkName>
+                    <spinDirection>cw</spinDirection>
+                    <timeConstantUp>${time_constant_up}</timeConstantUp>
+                    <timeConstantDown>${time_constant_down}</timeConstantDown>
+                    <minRotVelocity>${min_rot_velocity}</minRotVelocity>
+                    <maxRotVelocity>${max_rot_velocity}</maxRotVelocity>
+                    <thrustConstant>${motor_constant}</thrustConstant>
+                    <momentConstant>${moment_constant}</momentConstant>
+                    <rotorDragCoefficient>${rotor_drag_coefficient}</rotorDragCoefficient>
+                    <rollingMomentCoefficient>${rolling_moment_coefficient}</rollingMomentCoefficient>
+                    <rotorVelocitySlowdownSim>${rotor_velocity_slowdown_sim}</rotorVelocitySlowdownSim>
+                </rotor>
+                <rotor>
+                    <jointName>rear_rotor_joint</jointName>
+                    <linkName>rear_rotor</linkName>
+                    <spinDirection>ccw</spinDirection>
+                    <timeConstantUp>${time_constant_up}</timeConstantUp>
+                    <timeConstantDown>${time_constant_down}</timeConstantDown>
+                    <minRotVelocity>${min_rot_velocity}</minRotVelocity>
+                    <maxRotVelocity>${max_rot_velocity}</maxRotVelocity>
+                    <thrustConstant>${motor_constant}</thrustConstant>
+                    <momentConstant>${moment_constant}</momentConstant>
+                    <rotorDragCoefficient>${rotor_drag_coefficient}</rotorDragCoefficient>
+                    <rollingMomentCoefficient>${rolling_moment_coefficient}</rollingMomentCoefficient>
+                    <rotorVelocitySlowdownSim>${rotor_velocity_slowdown_sim}</rotorVelocitySlowdownSim>
+                </rotor>
+            </rotors>
+            <servos>
+                <servo>
+                    <jointName>${namespace}/tilt_wing_servo_0_revolutejoint</jointName>
+                    <spinDirection>ccw</spinDirection>
+                    <controlMode>${tilt_control_mode}</controlMode>
+                    <maxRotVelocity>${10}</maxRotVelocity>
+                    <minRotPosition>${-pi*6}</minRotPosition>
+                    <maxRotPosition>${pi*6}</maxRotPosition>
+                    <zeroOffset>${servo_zero_offset}</zeroOffset>
+                    <joint_control_pid>
+                        <p>${p_gain}</p>
+                        <i>${i_gain}</i>
+                        <d>${d_gain}</d>
+                        <iMax>1.0</iMax>
+                        <iMin>-1.0</iMin>
+                        <cmdMax>2.0</cmdMax>
+                        <cmdMin>-2.0</cmdMin>
+                    </joint_control_pid>
+                </servo>
+                <servo>
+                    <jointName>${namespace}/tilt_wing_servo_1_revolutejoint</jointName>
+                    <spinDirection>ccw</spinDirection>
+                    <controlMode>${tilt_control_mode}</controlMode>
+                    <maxRotVelocity>${10}</maxRotVelocity>
+                    <minRotPosition>${-pi*6}</minRotPosition>
+                    <maxRotPosition>${pi*6}</maxRotPosition>
+                    <zeroOffset>${servo_zero_offset}</zeroOffset>
+                    <joint_control_pid>
+                        <p>${p_gain}</p>
+                        <i>${i_gain}</i>
+                        <d>${d_gain}</d>
+                        <iMax>1.0</iMax>
+                        <iMin>-1.0</iMin>
+                        <cmdMax>2.0</cmdMax>
+                        <cmdMin>-2.0</cmdMin>
+                    </joint_control_pid>
+                </servo>
+                <servo>
+                    <jointName>${namespace}/motor_tilt_mechanism_servo_0_revolutejoint</jointName>
+                    <spinDirection>ccw</spinDirection>
+                    <controlMode>${tilt_control_mode}</controlMode>
+                    <maxRotVelocity>${10}</maxRotVelocity>
+                    <minRotPosition>${-pi*6}</minRotPosition>
+                    <maxRotPosition>${pi*6}</maxRotPosition>
+                    <zeroOffset>${servo_zero_offset}</zeroOffset>
+                    <joint_control_pid>
+                        <p>${p_gain}</p>
+                        <i>${i_gain}</i>
+                        <d>${d_gain}</d>
+                        <iMax>1.0</iMax>
+                        <iMin>-1.0</iMin>
+                        <cmdMax>2.0</cmdMax>
+                        <cmdMin>-2.0</cmdMin>
+                    </joint_control_pid>
+                </servo>
+                <servo>
+                    <jointName>${namespace}/motor_tilt_mechanism_servo_1_revolutejoint</jointName>
+                    <spinDirection>ccw</spinDirection>
+                    <controlMode>${tilt_control_mode}</controlMode>
+                    <maxRotVelocity>${10}</maxRotVelocity>
+                    <minRotPosition>${-pi*6}</minRotPosition>
+                    <maxRotPosition>${pi*6}</maxRotPosition>
+                    <zeroOffset>${servo_zero_offset}</zeroOffset>
+                    <joint_control_pid>
+                        <p>${p_gain}</p>
+                        <i>${i_gain}</i>
+                        <d>${d_gain}</d>
+                        <iMax>1.0</iMax>
+                        <iMin>-1.0</iMin>
+                        <cmdMax>2.0</cmdMax>
+                        <cmdMin>-2.0</cmdMin>
+                    </joint_control_pid>
+                </servo>
+            </servos>
+        </plugin>
+    </gazebo>
 </robot>

File: rotors_description/urdf/soliro_base.xacro (robot description, xacro)
@@ -3,5 +3,5 @@
     <xacro:include filename="$(find rotors_description)/urdf/component_snippets.xacro"/>
     <xacro:property name="mounting_roll" value="$(arg model_roll)" />
-    <!-- Instantiate OMAV "mechanics". -->
+    <!-- Instantiate Soliro "mechanics". -->
     <xacro:include filename="$(find rotors_description)/urdf/soliro.xacro"/>
     <xacro:include filename="$(find rotors_description)/urdf/soliro_actuators.xacro"/>
