Commit message: wip

File: rotors_description/urdf/soliro_actuators.xacro (robot description, xacro)
@@ -74,6 +74,6 @@
                     <controlMode>${tilt_control_mode}</controlMode>
                     <maxRotVelocity>${10}</maxRotVelocity>
-                    <minRotPosition>${-pi*6}</minRotPosition>
-                    <maxRotPosition>${pi*6}</maxRotPosition>
+                    <minRotPosition>${-pi}</minRotPosition>
+                    <maxRotPosition>${pi}</maxRotPosition>
                     <zeroOffset>${servo_zero_offset}</zeroOffset>
                     <joint_control_pid>
@@ -92,6 +92,6 @@
                     <controlMode>${tilt_control_mode}</controlMode>
                     <maxRotVelocity>${10}</maxRotVelocity>
-                    <minRotPosition>${-pi*6}</minRotPosition>
-                    <maxRotPosition>${pi*6}</maxRotPosition>
+                    <minRotPosition>${-pi}</minRotPosition>
+                    <maxRotPosition>${pi}</maxRotPosition>
                     <zeroOffset>${servo_zero_offset}</zeroOffset>
                     <joint_control_pid>
@@ -110,6 +110,6 @@
                     <controlMode>${tilt_control_mode}</controlMode>
                     <maxRotVelocity>${10}</maxRotVelocity>
-                    <minRotPosition>${-pi*6}</minRotPosition>
-                    <maxRotPosition>${pi*6}</maxRotPosition>
+                    <minRotPosition>${-pi/16}</minRotPosition>
+                    <maxRotPosition>${pi/16}</maxRotPosition>
                     <zeroOffset>${servo_zero_offset}</zeroOffset>
                     <joint_control_pid>
@@ -128,6 +128,6 @@
                     <controlMode>${tilt_control_mode}</controlMode>
                     <maxRotVelocity>${10}</maxRotVelocity>
-                    <minRotPosition>${-pi*6}</minRotPosition>
-                    <maxRotPosition>${pi*6}</maxRotPosition>
+                    <minRotPosition>${-pi/16}</minRotPosition>
+                    <maxRotPosition>${pi/16}</maxRotPosition>
                     <zeroOffset>${servo_zero_offset}</zeroOffset>
                     <joint_control_pid>

File: rotors_description/urdf/soliro_base.xacro (robot description, xacro)
@@ -39,5 +39,5 @@
                 wait_to_record_bag="$(arg wait_to_record_bag)"/>
     </xacro:if>
-    <!-- Add odometry. -->
-    <xacro:include filename="$(find rotors_description)/urdf/odometry_sensor_smooth.xacro"/>
+<!--    &lt;!&ndash; Add odometry. &ndash;&gt;-->
+<!--    <xacro:include filename="$(find rotors_description)/urdf/odometry_sensor_smooth.xacro"/>-->
 </robot>

File: rotors_description/urdf/soliro_snippets.xacro (robot description, xacro)
@@ -76,5 +76,5 @@
         <!-- Wing (wing_number: 0=right, 1=left)-->
         <joint name="${robot_namespace}/tilt_wing_servo_${wing_number}_revolutejoint" type="revolute">
-            <limit lower="-${pi}" upper="${pi}" effort="0" velocity="0"/>
+            <limit lower="-${pi}" upper="${pi}" effort="1000" velocity="1000"/>
             <xacro:if value="${wing_number}">
                 <origin xyz="0 0 0" rpy="0 0 0"/>
@@ -120,5 +120,5 @@
             <axis xyz="0 0 1"/>
             <!-- TODO check effort and velocity -->
-            <limit lower="-${pi/16}" upper="${pi/16}" effort="0" velocity="0"/>
+            <limit lower="-${pi/16}" upper="${pi/16}" effort="1000" velocity="1000"/>
             <parent link="${namespace}/tilt_wing_${wing_number}"/>
             <child link="${namespace}/motor_tilt_mechanism_${wing_number}"/>
