Commit message: Fixed wrong motor allocation (left and right was mixed up)

File: rotors_description/urdf/soliro_snippets.xacro (robot description, xacro)
@@ -77,10 +77,5 @@
         <joint name="${robot_namespace}/tilt_wing_servo_${wing_number}_revolutejoint" type="revolute">
             <limit lower="-${pi}" upper="${pi}" effort="1000" velocity="1000"/>
-            <xacro:if value="${wing_number}">
-                <origin xyz="0 0 0" rpy="0 0 0"/>
-            </xacro:if>
-            <xacro:unless value="${wing_number}">
-                <origin xyz="0 0 0" rpy="0 0 0"/>
-            </xacro:unless>
+            <origin xyz="0 0 0" rpy="0 0 0"/>
             <axis xyz="0 1 0"/>
             <parent link="${parent}"/>
@@ -97,8 +92,8 @@
             <visual>
                 <xacro:if value="${wing_number}">
-                    <origin xyz="0 0 0" rpy="0 0 0"/>
+                    <origin xyz="0 0 0" rpy="${pi} 0 0"/>
                 </xacro:if>
                 <xacro:unless value="${wing_number}">
-                    <origin xyz="0 0 0" rpy="${pi} 0 0"/>
+                    <origin xyz="0 0 0" rpy="0 0 0"/>
                 </xacro:unless>
                 <geometry>
